Commit message: velodyne demo

File: wpv4_bringup/urdf/wpv4.urdf (robot description, URDF)
Before this commit: robot WPV4, 10 links, 9 joints
Links:
- removed link velo_link
- added link velodyne; visual cylinder length=0.00 radius=0.00
Joints:
- joint velodyne_joint: child velo_link -> velodyne; origin xyz=0.2 0 1.7 rpy=0 0 0 -> xyz=0.3 0 0.3 rpy=0 0 0
