Commit message: add trackbars for wpm2

File: wpv4_bringup/urdf/wpv4_wpm2.urdf (robot description, URDF)
Before this commit: robot WPV4_WPM2, 21 links, 20 joints
Links:
- removed link velo_link
- added link velodyne; visual cylinder length=0.00 radius=0.00
- link laser: mass 10 -> None; geometry visual cylinder length=0 radius=0
- link lb_wheel: mass 10 -> None; geometry visual mesh filename=package://wpv4_bringup/meshes/wheel.dae scale=1 1 1
- link lf_wheel: mass 10 -> None; geometry visual mesh filename=package://wpv4_bringup/meshes/wheel.dae scale=1 1 1
- link rb_wheel: mass 10 -> None; geometry visual mesh filename=package://wpv4_bringup/meshes/wheel.dae scale=1 1 1
- link rf_wheel: mass 10 -> None; geometry visual mesh filename=package://wpv4_bringup/meshes/wheel.dae scale=1 1 1
Joints:
- joint base_to_lb_wheal: axis 0 1 0 -> (none); type continuous -> fixed
- joint base_to_lf_wheal: axis 0 1 0 -> (none); type continuous -> fixed
- joint base_to_rb_wheal: axis 0 -1 0 -> (none); type continuous -> fixed
- joint base_to_rf_wheal: axis 0 -1 0 -> (none); type continuous -> fixed
- joint laser_joint: origin xyz=0.2 0 0 rpy=0 0 0 -> xyz=0.32 0 0.2 rpy=0 0 0
- joint velodyne_joint: child velo_link -> velodyne; origin xyz=0.2 0 1.7 rpy=0 0 0 -> xyz=0.32 0 0.2 rpy=0 0 0

Commit message: add kinect_test

File: wpv4_bringup/urdf/wpv4_wpm2.urdf (robot description, URDF)
Before this commit: robot WPV4_WPM2, 21 links, 20 joints
Links:
- added link kinect2_left_rot; visual cylinder length=0.6 radius=0.01
- added link kinect2_right_rot; visual cylinder length=0.6 radius=0.01
- link kinect2_ir_optical_frame: geometry visual box size=.25 .04 .07
Joints:
- added joint kinect_left: type fixed, parent kinect2_dock, child kinect2_left_rot, origin xyz=0 0.04 -0.3 rpy=0 0 0
- added joint kinect_right: type fixed, parent kinect2_dock, child kinect2_right_rot, origin xyz=0 -0.04 -0.3 rpy=0 0 0
- joint kinect_height: origin xyz=0.174 0 0 rpy=0 -1.5707963 0 -> xyz=0.1 0 0 rpy=0 -1.5707963 0
